Commit message: Add files via upload

File: urdf/selfbalancerobot.urdf (robot description, URDF)
Before this commit: robot selfbalancerobot, 5 links, 4 joints
Links:
- link left_wheeL_link: geometry collision cylinder length=0.01 radius=0.1; visual mesh filename=package://selfbalancerobot/meshes/left_wheeL_link.STL
- link right_wheel_link: geometry collision cylinder length=0.01 radius=0.1; visual mesh filename=package://selfbalancerobot/meshes/right_wheel_link.STL
